Commit message: Getting the robot to move

File: description/robot.urdf.xacro (robot description, xacro)
@@ -2,3 +2,4 @@
 <robot xmlns:xacro="http://www.ros.org/wiki/xacro"  name="robot">
     <xacro:include filename="robot_core.xacro" />
+    <xacro:include filename="gazebo_control.xacro"/>
 </robot>

File: description/robot_core.xacro (robot description, xacro)
@@ -42,4 +42,7 @@
         </xacro:inertial_box>
     </link>
+    <gazebo reference ="chassis">
+        <material> Gazebe/White </material>
+    </gazebo>
     <!-- LEFT WHEEL LINK -->
     <joint name="left_wheel_joint" type="continuous">
@@ -65,4 +68,7 @@
         </xacro:inertial_cylinder>
     </link>
+    <gazebo reference ="left_wheel">
+        <material> Gazebo/Blue </material>
+    </gazebo>
     <!-- RIGHT WHEEL LINK -->
     <joint name="right_wheel_joint" type="continuous">
@@ -88,4 +94,7 @@
         </xacro:inertial_cylinder>
     </link>
+    <gazebo reference ="right_wheel">
+        <material> Gazebo/Blue </material>
+    </gazebo>
     <!--CASTER WHEEL-->
     <joint name="caster_wheel_joint" type="fixed">
@@ -110,3 +119,8 @@
         </xacro:inertial_sphere>
     </link>
+    <gazebo reference ="caster_wheel">
+        <material> Gazebo/Black </material>
+        <mu1 value="0.001"/>
+        <mu2 value="0.001"/>
+    </gazebo>
 </robot>

Commit message: added lidar and camera sensor

File: description/robot.urdf.xacro (robot description, xacro)
@@ -3,3 +3,5 @@
     <xacro:include filename="robot_core.xacro" />
     <xacro:include filename="gazebo_control.xacro"/>
+    <xacro:include filename="lidar.xacro"/>
+    <xacro:include filename="camera.xacro"/>
 </robot>

File: description/robot_core.xacro (robot description, xacro)
@@ -13,4 +13,7 @@
     <material  name="black">
         <color rgba="0 0 0 1"/>
+    </material>
+    <material  name="red">
+        <color rgba="1 0 0 1"/>
     </material>
     <!-- orientation is front = +x left = +y up = +z-->
